Commit message: Update vx300s_macro.xacro

File: vx300s_description/urdf/vx300s_macro.xacro (robot description, xacro)
@@ -202,5 +202,5 @@
     <joint name="${prefix}wrist_rotate" type="revolute">
       <axis xyz="1 0 0" />
-      <limit effort="1" lower="${-pi + pi_offset}" upper="${pi - pi_offset}" velocity="${pi}" />
+      <limit effort="1" lower="${-pi/2 + pi_offset}" upper="${pi/2 - pi_offset}" velocity="${pi}" />
       <origin rpy="0 0 0" xyz="0.069744 0 0" />
       <parent link="${prefix}wrist_link" />
